File: Kicad/kicad_ampli.sch (KiCad schematic (older format))
At the start: 108 parts, among them J1 AudioJack2, J2 Screw_Terminal_01x02, J3 Conn_01x01_Male, J3(GND)1 Conn_01x01_Male, J4 Conn_01x01_Male, J5 Conn_01x01_Male, J6 Conn_01x01_Male, J7 Conn_01x01_Male, J8 Conn_01x01_Male, Q1 BC546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

Commit message: Kicad_final
Parts:
- added Ccomp2, Ccomp3: 220, symbol Device:C
- added R9: 100, symbol Device:R
- added R?: R, symbol Device:R
- renumbered R9 to RV2
Connections:
- net at C12.1, C8.1, D7.2 (A)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: now also Ccomp2.1
- net at C13.2, C9.1, D2.1 (K)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: now also Ccomp3.2
- net at C7.1, D4.2 (A), Q19.3 (C)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: now also R9.2; no longer Q13.3 (B)
- net at C7.2, D3.1 (K), Q18.3 (C)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: now also R?.2; no longer Q10.3 (B)
- net at Q12.1 (E), Q14.1 (B), R17.1: now also Ccomp2.2
- net at Q13.1 (E), Q15.1 (B), R18.1: now also Q15.3 (E), Q19.2 (B), R20.1
- net at Q11.1 (E), Q17.1 (B), R16.2: now also Ccomp3.1
- new net: Q13.3 (B), R9.1
- new net: Q10.3 (B), R?.1
Other:
- moved on the sheet: C7, D6, Q10, Q11, Q17, Q18, Q19, R16, R18, R19
